File: hardware/stm32-plant-monitor.kicad_sch (KiCad schematic)
At the start: 11 parts, among them J1 Soil_Sensor, J2 BH1750, J3 SD_Card, J4 Pump_Relay, J5 EXT_5V, J6 Relay_out, J7 Pump, J8 Grow_LED, U1 NUCLEO64-F411RE

Commit message: Chore: pump relay open drain (#10)
* chore: 펌프 릴레이 핀 오픈 드레인 설정 변경

원인: Low 트리거 PNP 모듈 (VCC 5V)에 3.3V HIGH를 주면 릴레이가 꺼지지 않음

* docs: 회로도 릴레이 입력 핀 순서 수정 및 풀업 추가
Parts:
- added R2: 10k, symbol Device:R
Connections:
- net +5V: now also J4.3 (Pin_3), R2.1; no longer J4.1 (Pin_1)
- net PUMP_RELAY: now also J4.1 (Pin_1), R2.2; no longer J4.3 (Pin_3)
Other:
- note added: "[ASSUMPTION] Connector pin order follows common modules (web search) - verify against board silkscreen J1 HW-390: GND / VCC / AOUT (work report 2026-10-12) J2 GY-302: VCC / GND / SCL / SDA / ADDR, on-board I2C pull-ups, ADDR=GND -> 0x23 J3 microSD (Catalex type): GND / VCC / MISO / MOSI / SCK / CS, VCC 5V (on-board 3.3V LDO) J4 relay input: IN / GND / VCC(5V) (verified 2026-10-14), S8550 PNP low-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"
- note removed: "[ASSUMPTION] Connector pin order follows common modules (web search) - verify against board silkscreen J1 HW-390: GND / VCC / AOUT (work report 2026-10-12) J2 GY-302: VCC / GND / SCL / SDA / ADDR, on-board I2C pull-ups, ADDR=GND -> 0x23 J3 microSD (Catalex type): GND / VCC / MISO / MOSI / SCK / CS, VCC 5V (on-board 3.3V LDO) J4 relay input: DC+ / DC- / IN, 5V module - check OFF behavior with 3.3V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"
Changed lines of the file:
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@@
 		)
 	)
-	(text "[ASSUMPTION] Connector pin order follows common modules (web search) - verify against board silkscreen\nJ1 HW-390: GND / VCC / AOUT (work report 2026-10-12)\nJ2 GY-302: VCC / GND / SCL / SDA / ADDR, on-board I2C pull-ups, ADDR=GND -> 0x23\nJ3 microSD (Catalex type): GND / VCC / MISO / MOSI / SCK / CS, VCC 5V (on-board 3.3V LDO)\nJ4 relay input: DC+ / DC- / IN, 5V module - check OFF behavior with 3.3V IN\nJ6 relay contacts: NO / COM / NC (verify terminal order)"
+	(text "[ASSUMPTION] Connector pin order follows common modules (web search) - verify against board silkscreen\nJ1 HW-390: GND / VCC / AOUT (work report 2026-10-12)\nJ2 GY-302: VCC / GND / SCL / SDA / ADDR, on-board I2C pull-ups, ADDR=GND -> 0x23\nJ3 microSD (Catalex type): GND / VCC / MISO / MOSI / SCK / CS, VCC 5V (on-board 3.3V LDO)\nJ4 relay input: IN / GND / VCC(5V) (verified 2026-10-14), S8550 PNP low-trigger:\nPA8 open-drain + R2 10k pull-up to +5V (3.3V HIGH cannot turn relay OFF)\nJ6 relay contacts: NO / COM / NC (verify terminal order)"
 		(exclude_from_sim no)
 		(at 175.26 30.48 0)
@@
 			(justify left bottom)
 		)
+	)
+	(junction
+		(at 154.94 107.95)
+		(diameter 0)
+		(color 0 0 0 0)
 	)
 	(no_connect
@@
 	(wire
 		(pts
-			(xy 158.75 93.98) (xy 151.13 93.98)
+			(xy 154.94 105.41) (xy 154.94 107.95)
 		)
 		(stroke
@@
 	(wire
 		(pts
-			(xy 160.02 60.96) (xy 152.4 60.96)
+			(xy 158.75 93.98) (xy 151.13 93.98)
 		)
 		(stroke
@@
 	(wire
 		(pts
-			(xy 158.75 143.51) (xy 151.13 143.51)
+			(xy 160.02 60.96) (xy 152.4 60.96)
 		)
 		(stroke
@@
 	(wire
 		(pts
-			(xy 81.28 175.26) (xy 91.44 175.26)
+			(xy 158.75 143.51) (xy 151.13 143.51)
 		)
 		(stroke
@@
 	(wire
 		(pts
-			(xy 160.02 58.42) (xy 152.4 58.42)
+			(xy 81.28 175.26) (xy 91.44 175.26)
 		)
 		(stroke
@@
 	(wire
 		(pts
-			(xy 87.63 53.34) (xy 87.63 50.8)
+			(xy 160.02 58.42) (xy 152.4 58.42)
 		)
 		(stroke
@@
 	(wire
 		(pts
-			(xy 158.75 86.36) (xy 151.13 86.36)
+			(xy 87.63 53.34) (xy 87.63 50.8)
 		)
 		(stroke
@@
 	(wire
 		(pts
-			(xy 158.75 129.54) (xy 151.13 129.54)
+			(xy 158.75 86.36) (xy 151.13 86.36)
 		)
 		(stroke
@@
 	(wire
 		(pts
-			(xy 147.32 179.07) (xy 158.75 179.07)
+			(xy 158.75 129.54) (xy 151.13 129.54)
 		)
 		(stroke
@@
 	(wire
 		(pts
-			(xy 158.75 113.03) (xy 151.13 113.03)
+			(xy 147.32 179.07) (xy 158.75 179.07)
 		)
 		(stroke
@@
 	(wire
 		(pts
-			(xy 158.75 127) (xy 151.13 127)
+			(xy 158.75 107.95) (xy 151.13 107.95)
 		)
 		(stroke
@@
 	(wire
 		(pts
-			(xy 158.75 165.1) (xy 151.13 165.1)
+			(xy 158.75 127) (xy 151.13 127)
 		)
 		(stroke
@@
 	(wire
 		(pts
-			(xy 158.75 146.05) (xy 151.13 146.05)
+			(xy 158.75 165.1) (xy 151.13 165.1)
 		)
 		(stroke
@@
 	(wire
 		(pts
-			(xy 158.75 91.44) (xy 151.13 91.44)
+			(xy 158.75 146.05) (xy 151.13 146.05)
 		)
 		(stroke
@@
 	(wire
 		(pts
-			(xy 58.42 175.26) (xy 68.58 175.26)
+			(xy 158.75 91.44) (xy 151.13 91.44)
 		)
 		(stroke
@@
 	(wire
 		(pts
-			(xy 158.75 162.56) (xy 151.13 162.56)
+			(xy 58.42 175.26) (xy 68.58 175.26)
 		)
 		(stroke
@@
 	(wire
 		(pts
-			(xy 158.75 88.9) (xy 151.13 88.9)
+			(xy 158.75 162.56) (xy 151.13 162.56)
 		)
 		(stroke
@@
 	(wire
 		(pts
-			(xy 35.56 175.26) (xy 45.72 175.26)
+			(xy 158.75 88.9) (xy 151.13 88.9)
 		)
 		(stroke
@@
 	(wire
 		(pts
-			(xy 87.63 50.8) (xy 92.71 50.8)
+			(xy 35.56 175.26) (xy 45.72 175.26)
 		)
 		(stroke
@@
 		)
 	)
+	(wire
+		(pts
+			(xy 87.63 50.8) (xy 92.71 50.8)
+		)
+		(stroke
+			(width 0)
+			(type default)
+		)
+	)
 	(label "SPI_SCK"
 		(at 120.65 139.7 0)
@@
 	)
 	(label "PUMP_RELAY"
-		(at 151.13 113.03 180)
+		(at 151.13 107.95 180)
 		(effects
 			(font
@@
 	)
 	(symbol
+		(lib_id "power:+5V")
+		(at 154.94 97.79 90)
+		(unit 1)
+		(body_style 1)
+		(exclude_from_sim no)
+		(in_bom yes)
+		(on_board yes)
+		(in_pos_files yes)
+		(dnp no)
+		(property "Reference" "#PWR045"
+			(at 154.94 97.79 90)
+			(hide yes)
+			(show_name no)
+			(do_not_autoplace no)
+			(effects
+				(font
+					(size 1.27 1.27)
+				)
+			)
+		)
+		(property "Value" "+5V"
+			(at 149.99 97.79 90)
+			(show_name no)
+			(do_not_autoplace no)
+			(effects
+				(font
+					(size 1.27 1.27)
+				)
+			)
+		)
+		(property "Footprint" ""
+			(at 154.94 97.79 0)
+			(hide yes)
+			(show_name no)
+			(do_not_autoplace no)
+			(effects
+				(font
+					(size 1.27 1.27)
+				)
+			)
+		)
+		(property "Datasheet" ""
+			(at 154.94 97.79 0)
+			(hide yes)
+			(show_name no)
+			(do_not_autoplace no)
+			(effects
+				(font
+					(size 1.27 1.27)
+				)
+			)
+		)
+		(property "Description" "Power symbol creates a global label with name \"+5V\""
+			(at 154.94 97.79 0)
+			(hide yes)
+			(show_name no)
+			(do_not_autoplace no)
+			(effects
+				(font
+					(size 1.27 1.27)
+				)
+			)
+		)
+		(pin "1"
+		)
+		(instances
+			(project "stm32-plant-monitor"
+				(path "/8c11d841-cc40-4395-990f-fa64c6c3dd44"
+					(reference "#PWR045")
+					(unit 1)
+				)
+			)
+		)
+	)
+	(symbol
 		(lib_id "power:GND")
 		(at 100.33 154.94 0)
@@
 	(symbol
 		(lib_id "power:+5V")
-		(at 158.75 107.95 90)
+		(at 158.75 113.03 90)
 		(unit 1)
 		(body_style 1)
@@
 		(dnp no)
 		(property "Reference" "#PWR038"
-			(at 158.75 107.95 90)
+			(at 158.75 113.03 90)
 			(hide yes)
 			(show_name no)
@@
 		)
 		(property "Value" "+5V"
-			(at 153.8 107.95 90)
+			(at 153.8 113.03 90)
 			(show_name no)
 			(do_not_autoplace no)
@@
 		)
 		(property "Footprint" ""
-			(at 158.75 107.95 0)
+			(at 158.75 113.03 0)
 			(hide yes)
 			(show_name no)
@@
 		)
 		(property "Datasheet" ""
-			(at 158.75 107.95 0)
+			(at 158.75 113.03 0)
 			(hide yes)
 			(show_name no)
@@
 		)
 		(property "Description" "Power symbol creates a global label with name \"+5V\""
-			(at 158.75 107.95 0)
+			(at 158.75 113.03 0)
 			(hide yes)
 			(show_name no)
@@
 					(unit 1)
 				)
+			)
+		)
+	)
+	(symbol
+		(lib_id "Device:R")
+		(at 154.94 101.6 0)
+		(unit 1)
+		(body_style 1)
+		(exclude_from_sim no)
+		(in_bom yes)
+		(on_board yes)
+		(in_pos_files yes)
+		(dnp no)
+		(property "Reference" "R2"
+			(at 156.972 100.33 0)
+			(show_name no)
+			(do_not_autoplace no)
+			(effects
+				(font
+					(size 1.27 1.27)
+				)
+				(justify left)
+			)
+		)
+		(property "Value" "10k"
+			(at 156.972 102.87 0)
+			(show_name no)
+			(do_not_autoplace no)
+			(effects
+				(font
+					(size 1.27 1.27)
+				)
+				(justify left)
+			)
+		)
+		(property "Footprint" ""
+			(at 153.162 101.6 90)
+			(hide yes)
+			(show_name no)
+			(do_not_autoplace no)
+			(effects
+				(font
+					(size 1.27 1.27)
+				)
+			)
+		)
+		(property "Datasheet" "~"
+			(at 154.94 101.6 0)
+			(hide yes)
+			(show_name no)
+			(do_not_autoplace no)
+			(effects
+				(font
+					(size 1.27 1.27)
+				)
+			)
+		)
+		(property "Description" "Resistor"
+			(at 154.94 101.6 0)
+			(hide yes)
+			(show_name no)
+			(do_not_autoplace no)
+			(effects
+				(font
+					(size 1.27 1.27)
+				)
+			)
+		)
+		(pin "1"
+		)
+		(pin "2"
+		)
+		(instances
+			(project "stm32-plant-monitor"
+				(path "/8c11d841-cc40-4395-990f-fa64c6c3dd44"
+					(reference "R2")
+					(unit 1)
+				)
